File: hardware/ledbarhack/PentaFnord_LedBar_0_91r.sch (EAGLE design)
At the start: 113 parts, among them IC1 MEGA8-AI, IC2 MAX487, IC3 78L05, Q1 BSS138, Q2 BSS138, Q3 BSS138, Q4 BSS138, Q5 BSS138, SW1 MCMT5-F-VADAPTED_FOOTPRINT, U1 NICHIA_NSSL157T-H3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

Commit message: routing done
Parts:
- A_L, B_L, C_L, D_L: value WIREPADSMD1,27-254 -> WIREPADSMD2,54-5,08; device wirepad:WIREPADSMD1,27-254 -> wirepad:WIREPADSMD2,54-5,08
Connections:
- net SPARE_B1: now also IC1.PB1(OC1A)
- net VCC: now also JP3A.2
Changed lines of the file:
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@@
 <part name="A_R" library="wirepad" deviceset="WIREPAD" device="SMD1,27-254" value=""/>
 <part name="GND_L" library="wirepad" deviceset="WIREPAD" device="SMD2,54-5,08" value=""/>
-<part name="B_L" library="wirepad" deviceset="WIREPAD" device="SMD1,27-254" value=""/>
+<part name="B_L" library="wirepad" deviceset="WIREPAD" device="SMD2,54-5,08" value=""/>
 <part name="+18_L" library="wirepad" deviceset="WIREPAD" device="SMD2,54-5,08" value=""/>
-<part name="A_L" library="wirepad" deviceset="WIREPAD" device="SMD1,27-254" value=""/>
+<part name="A_L" library="wirepad" deviceset="WIREPAD" device="SMD2,54-5,08" value=""/>
 <part name="GND6" library="supply1" deviceset="GND" device=""/>
 <part name="P+10" library="supply1" deviceset="VCC" device=""/>
@@
 <part name="PAD4" library="wirepad" deviceset="WIREPAD" device="SMD1,27-254"/>
 <part name="C3" library="rcl" deviceset="CPOL-EU" device="SMCD" value="10uF/25V"/>
-<part name="D_L" library="wirepad" deviceset="WIREPAD" device="SMD1,27-254"/>
-<part name="C_L" library="wirepad" deviceset="WIREPAD" device="SMD1,27-254"/>
+<part name="D_L" library="wirepad" deviceset="WIREPAD" device="SMD2,54-5,08"/>
+<part name="C_L" library="wirepad" deviceset="WIREPAD" device="SMD2,54-5,08"/>
 <part name="C" library="wirepad" deviceset="WIREPAD" device="SMD1,27-254"/>
 <part name="D" library="wirepad" deviceset="WIREPAD" device="SMD1,27-254"/>
@@
 <part name="Q4" library="transistor-small-signal" deviceset="BSS123" device="" value="BSS138"/>
 <part name="Q5" library="transistor-small-signal" deviceset="BSS123" device="" value="BSS138"/>
+<part name="P+2" library="supply1" deviceset="VCC" device=""/>
 </parts>
 <sheets>
@@
 <attribute name="VALUE" x="-1.778" y="46.863" size="1.778" layer="96" rot="MR270"/>
 </instance>
+<instance part="P+2" gate="VCC" x="182.88" y="132.08"/>
 </instances>
 <busses>
@@
 <junction x="-91.44" y="43.18"/>
 </segment>
+<segment>
+<pinref part="JP3A" gate="A" pin="2"/>
+<wire x1="175.26" y1="124.46" x2="182.88" y2="124.46" width="0.1524" layer="91"/>
+<wire x1="182.88" y1="124.46" x2="182.88" y2="129.54" width="0.1524" layer="91"/>
+<pinref part="P+2" gate="VCC" pin="VCC"/>
+<label x="185.42" y="127" size="1.778" layer="95"/>
+</segment>
 </net>
 <net name="SCK" class="0">
@@
 <wire x1="162.56" y1="121.92" x2="167.64" y2="121.92" width="0.1524" layer="91"/>
 <pinref part="JP3A" gate="A" pin="3"/>
+<label x="157.48" y="121.92" size="1.778" layer="95"/>
 </segment>
 </net>
@@
 <wire x1="-25.4" y1="45.72" x2="-27.94" y2="45.72" width="0.1524" layer="91"/>
 <pinref part="IC1" gate="G$1" pin="PC3(ADC3)"/>
+<wire x1="-25.4" y1="45.72" x2="-17.78" y2="45.72" width="0.1524" layer="91"/>
 </segment>
 <segment>
@@
 <pinref part="SW1" gate="G$1" pin="DUMMY"/>
 </segment>
-</net>
+<segment>
+<pinref part="IC1" gate="G$1" pin="PB1(OC1A)"/>
+<wire x1="-25.4" y1="5.08" x2="-15.24" y2="5.08" width="0.1524" layer="91"/>
+<wire x1="-15.24" y1="5.08" x2="-15.24" y2="2.54" width="0.1524" layer="91"/>
+</segment>
+</net>
